File: boards/Xduino6.0/Xduino6.0.brd (EAGLE design)
At the start: 40.2 x 61.1 mm, 21 parts, among them J1 JACK.65MM

Commit message: Download Files
New Xduino6 Files
Connections:
- removed net N$3: C5.2, IC1.2, J1.PIN
- net EXTVCC: now also C5.2, IC1.2, J1.PIN; no longer J1.CONTACT
Routing:
- net EXTVCC: track 8.64 -> 25.2 mm
- net N$3: track 12.5 -> 0.00 mm
- net GND: track 212.5 -> 220.8 mm
Changed lines of the file:
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@@
 <wire x1="12.1158" y1="28.727" x2="12.1162" y2="28.7274" width="0.4064" layer="1"/>
 <contactref element="J1" pad="SHUNT"/>
-<wire x1="23.1394" y1="53.3732" x2="25.9588" y2="53.3732" width="0.4064" layer="1"/>
-<wire x1="25.9588" y1="53.3732" x2="26.1792" y2="53.3732" width="0.4064" layer="1"/>
-<wire x1="26.1792" y1="53.3732" x2="26.543" y2="53.0094" width="0.4064" layer="1"/>
 <wire x1="1.3462" y1="16.9418" x2="1.3462" y2="34.3916" width="0.4064" layer="1"/>
 <wire x1="36.2712" y1="5.2578" x2="36.2712" y2="9.881" width="0.4064" layer="1"/>
@@
 <wire x1="37.4396" y1="51.5566" x2="37.4102" y2="51.586" width="0.4064" layer="1"/>
 <wire x1="26.5934" y1="52.959" x2="26.543" y2="53.0094" width="0.4064" layer="1"/>
-<wire x1="26.3476" y1="52.9844" x2="25.9588" y2="53.3732" width="0.4064" layer="1"/>
 <wire x1="3.5056" y1="36.551" x2="1.3462" y2="34.3916" width="0.4064" layer="1"/>
 <wire x1="6.7056" y1="59.436" x2="18.4404" y2="59.436" width="0.4064" layer="1"/>
 <wire x1="18.4404" y1="59.436" x2="19.558" y2="58.3184" width="0.4064" layer="1"/>
 <wire x1="19.558" y1="58.3184" x2="19.6342" y2="53.0602" width="0.4064" layer="1"/>
-<wire x1="26.3476" y1="52.9844" x2="27.8384" y2="52.9844" width="0.4064" layer="1"/>
-<wire x1="27.8384" y1="52.9844" x2="28.4988" y2="52.324" width="0.4064" layer="1"/>
 <contactref element="C2" pad="1"/>
 <contactref element="JP1" pad="5"/>
@@
 <wire x1="35.2044" y1="45.2882" x2="36.2712" y2="45.2882" width="0.4064" layer="1"/>
 <wire x1="36.2712" y1="45.2882" x2="36.3728" y2="45.2374" width="0.4064" layer="1"/>
-<wire x1="36.3728" y1="45.2374" x2="36.2966" y2="47.5996" width="0.4064" layer="1"/>
 <wire x1="36.2966" y1="47.5996" x2="37.465" y2="48.768" width="0.4064" layer="1"/>
 <wire x1="37.465" y1="48.768" x2="37.465" y2="51.5312" width="0.4064" layer="1"/>
@@
 <wire x1="23.0886" y1="58.2676" x2="19.6088" y2="58.2676" width="0.4064" layer="1"/>
 <wire x1="19.6088" y1="58.2676" x2="19.558" y2="58.3184" width="0.4064" layer="1"/>
-<wire x1="28.4988" y1="52.324" x2="28.4988" y2="50.419" width="0.4064" layer="1"/>
-<wire x1="28.4988" y1="50.419" x2="29.2608" y2="49.657" width="0.4064" layer="1"/>
-<wire x1="29.2608" y1="49.657" x2="30.9626" y2="49.657" width="0.4064" layer="1"/>
-<wire x1="30.9626" y1="49.657" x2="32.8676" y2="51.562" width="0.4064" layer="1"/>
-<wire x1="32.8676" y1="51.562" x2="37.3862" y2="51.562" width="0.4064" layer="1"/>
-<wire x1="37.3862" y1="51.562" x2="37.4102" y2="51.586" width="0.4064" layer="1"/>
+<wire x1="37.4102" y1="51.586" x2="35.536" y2="51.586" width="0.4064" layer="1"/>
+<wire x1="35.536" y1="51.586" x2="33.528" y2="53.594" width="0.4064" layer="1"/>
+<wire x1="33.528" y1="53.594" x2="33.528" y2="59.3344" width="0.4064" layer="1"/>
+<wire x1="33.528" y1="59.3344" x2="32.4866" y2="60.3758" width="0.4064" layer="1"/>
+<wire x1="32.4866" y1="60.3758" x2="23.6474" y2="60.3758" width="0.4064" layer="1"/>
+<wire x1="23.6474" y1="60.3758" x2="23.0378" y2="59.7662" width="0.4064" layer="1"/>
+<wire x1="23.0378" y1="59.7662" x2="23.0378" y2="58.3184" width="0.4064" layer="1"/>
+<wire x1="23.0378" y1="58.3184" x2="23.0886" y2="58.2676" width="0.4064" layer="1"/>
+<wire x1="23.1394" y1="53.3732" x2="26.1792" y2="53.3732" width="0.4064" layer="1"/>
+<wire x1="26.1792" y1="53.3732" x2="26.543" y2="53.0094" width="0.4064" layer="1"/>
+<wire x1="36.2966" y1="47.5996" x2="36.2966" y2="45.3136" width="0.4064" layer="1"/>
+<wire x1="36.2966" y1="45.3136" x2="36.3728" y2="45.2374" width="0.4064" layer="1"/>
 </signal>
 <signal name="N$7">
@@
 <signal name="N$1">
 <wire x1="24.5364" y1="25.0698" x2="30.861" y2="25.0698" width="0.4064" layer="1"/>
-</signal>
-<signal name="N$3">
-<contactref element="IC1" pad="2"/>
-<contactref element="C5" pad="2"/>
-<contactref element="J1" pad="PIN"/>
-<wire x1="33.7281" y1="49.3522" x2="33.8959" y2="49.52" width="0.4064" layer="1"/>
-<wire x1="24.0894" y1="51.1732" x2="24.8998" y2="51.1732" width="0.4064" layer="1"/>
-<wire x1="24.8998" y1="51.1732" x2="25.8826" y2="50.1904" width="0.4064" layer="1"/>
-<wire x1="25.8826" y1="50.1904" x2="26.518" y2="50.1904" width="0.4064" layer="1"/>
-<wire x1="26.518" y1="50.1904" x2="26.543" y2="50.1654" width="0.4064" layer="1"/>
-<wire x1="26.543" y1="50.1654" x2="26.543" y2="48.895" width="0.4064" layer="1"/>
-<wire x1="26.543" y1="48.895" x2="27.1018" y2="48.3362" width="0.4064" layer="1"/>
-<wire x1="27.1018" y1="48.3362" x2="31.2674" y2="48.3362" width="0.4064" layer="1"/>
-<wire x1="31.2674" y1="48.3362" x2="32.4104" y2="49.4792" width="0.4064" layer="1"/>
-<wire x1="32.4104" y1="49.4792" x2="33.8551" y2="49.4792" width="0.4064" layer="1"/>
-<wire x1="33.8551" y1="49.4792" x2="33.8959" y2="49.52" width="0.4064" layer="1"/>
 </signal>
 <signal name="N$12">
@@
 <signal name="EXTVCC">
 <contactref element="JP6" pad="1"/>
-<contactref element="J1" pad="CONTACT"/>
-<wire x1="25.6286" y1="58.2676" x2="27.2796" y2="58.2676" width="0.4064" layer="1"/>
-<wire x1="27.2796" y1="58.2676" x2="28.0162" y2="57.531" width="0.4064" layer="1"/>
-<wire x1="28.0162" y1="57.531" x2="28.0162" y2="54.9312" width="0.4064" layer="1"/>
-<wire x1="28.0162" y1="54.9312" x2="30.3817" y2="52.5657" width="0.4064" layer="1"/>
+<contactref element="IC1" pad="2"/>
+<contactref element="C5" pad="2"/>
+<contactref element="J1" pad="PIN"/>
+<wire x1="33.7281" y1="49.3522" x2="33.8959" y2="49.52" width="0.4064" layer="1"/>
+<wire x1="24.0894" y1="51.1732" x2="24.8998" y2="51.1732" width="0.4064" layer="1"/>
+<wire x1="24.8998" y1="51.1732" x2="25.8826" y2="50.1904" width="0.4064" layer="1"/>
+<wire x1="25.8826" y1="50.1904" x2="26.518" y2="50.1904" width="0.4064" layer="1"/>
+<wire x1="26.518" y1="50.1904" x2="26.543" y2="50.1654" width="0.4064" layer="1"/>
+<wire x1="26.543" y1="50.1654" x2="29.9462" y2="50.1654" width="0.4064" layer="1"/>
+<wire x1="29.9462" y1="50.1654" x2="30.607" y2="49.5046" width="0.4064" layer="1"/>
+<wire x1="30.607" y1="49.5046" x2="33.8805" y2="49.5046" width="0.4064" layer="1"/>
+<wire x1="33.8805" y1="49.5046" x2="33.8959" y2="49.52" width="0.4064" layer="1"/>
+<wire x1="25.6286" y1="58.2676" x2="25.6286" y2="56.769" width="0.4064" layer="1"/>
+<wire x1="25.6286" y1="56.769" x2="27.5844" y2="54.8132" width="0.4064" layer="1"/>
+<wire x1="27.5844" y1="54.8132" x2="31.5214" y2="54.8132" width="0.4064" layer="1"/>
+<wire x1="31.5214" y1="54.8132" x2="32.385" y2="53.9496" width="0.4064" layer="1"/>
+<wire x1="32.385" y1="53.9496" x2="32.385" y2="51.0309" width="0.4064" layer="1"/>
+<wire x1="32.385" y1="51.0309" x2="33.8959" y2="49.52" width="0.4064" layer="1"/>
 </signal>
 </signals>
